Commit message: Functional urdf model loaded from github for OADK-D camera

File: husarion_workspace/pro3/rosbot_description/urdf/components/base_macro.urdf.xacro (robot description, xacro)
@@ -35,5 +35,7 @@
 					<geometry>
 						<!-- <mesh filename="${file_prefix}/urdf/models/${model}.stl" /> -->
-						<mesh filename="package://rosbot_description/meshes/${model}.stl" />
+						<!-- <mesh filename="package://depthai_descriptions/urdf/models/${model}.stl" /> -->
+						<!-- <mesh filename="package://ros_components_description/meshes/zed2i.stl" /> -->
+						<mesh filename="https://raw.githubusercontent.com/luxonis/depthai-ros/humble/depthai_descriptions/urdf/models/${model}.stl" />
 					</geometry>
 					<material name="mat">
@@ -49,5 +51,7 @@
 					<geometry>
 						<!-- <mesh filename="${file_prefix}/urdf/models/${model}.stl" /> -->
-						<mesh filename="package://rosbot_description/meshes/${model}.stl" />
+						<!-- <mesh filename="package://depthai_descriptions/urdf/models/${model}.stl" /> -->
+						<!-- <mesh filename="package://ros_components_description/meshes/zed2i.stl" /> -->
+						<mesh filename="https://raw.githubusercontent.com/luxonis/depthai-ros/humble/depthai_descriptions/urdf/models/${model}.stl" />
 					</geometry>
 					<material name="mat">
